File: Board Layout/BBQ_Blower.brd (EAGLE design)
At the start: 84.9 x 75.9 mm, 27 parts, among them IC1 MAX31855RASA+, IC2 MAX31855RASA+, IC3 MAX31855RASA+, J1 PCC-SMP-K-100-R-ROHS, J3 PCC-SMP-K-100-R-ROHS, J4 PCC-SMP-K-100-R-ROHS, Q1 BUZ10, Q2 BUZ10, U1 113990105

Commit message: moved header
Parts:
- moved D4 29.2 mm to (50.8, 78.5)
- moved D3 29.2 mm to (50.8, 74.2)
- moved M2 11.9 mm to (35.8, 75.7)
- moved M1 11.4 mm to (24.4, 75.7)
- moved PWR 1.02 mm to (60.7, 75.7)
Routing:
- net BLOWER1: track 42.7 -> 28.5 mm
- net VDD: track 73.7 -> 70.2 mm
- net BLOWER2: track 32.6 -> 33.8 mm
- net BLOWER_1: track 89.7 -> 89.0 mm
