File: Board Layout/BBQ_Blower.sch (EAGLE design)
At the start: 27 parts, among them IC1 MAX31855RASA+, IC2 MAX31855RASA+, IC3 MAX31855RASA+, J1 PCC-SMP-K-100-R-ROHS, J3 PCC-SMP-K-100-R-ROHS, J4 PCC-SMP-K-100-R-ROHS, Q1 BUZ10, Q2 BUZ10, U1 113990105

Commit message: re-arraging
Connections:
- removed net RELAY_1: U1.D2_-_GPIO4
- removed net RELAY_2: U1.D3_-_GPIO0
- new net DIO5: U$5.DIO5, U1.D11_-_GPIO9_/_SD_D2
- new net N$1: U1.RESV
- net D2: no longer U1.D11_-_GPIO9_/_SD_D2
- net D4: no longer U1.D4_-_GPIO2_/_TXD1
- net DIO0: now also U1.D2_-_GPIO4
- net DIO1: now also U1.D3_-_GPIO0
- net DIO2: now also U1.D4_-_GPIO2_/_TXD1
Other:
- moved on the sheet: C5, C6

Commit message: silk and wiring complete
Connections:
- removed net N$1: U1.RESV
- net 3V3: now also JP1.8, U1.VDD3V3(1); no longer JP1.10
- net CLK: now also U$5.SCK
- net DIO0: now also U1.D4_-_GPIO2_/_TXD1; no longer U1.D2_-_GPIO4
- net DIO2: now also U1.D2_-_GPIO4; no longer U1.D4_-_GPIO2_/_TXD1
- net EN: now also JP1.9; no longer JP1.8
- net RST: now also JP1.10, U1.RESV; no longer JP1.9
- net SCK: no longer U$5.SCK
Changed lines of the file:
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@@
 <attribute name="VALUE" x="208.0514" y="160.02" size="1.778" layer="96" rot="R90"/>
 </instance>
-<instance part="M2" gate="G$1" x="228.6" y="160.02" smashed="yes" rot="MR0"/>
+<instance part="M2" gate="G$1" x="223.52" y="154.94" smashed="yes" rot="MR0"/>
 <instance part="VDD_12V3" gate="G$1" x="205.74" y="170.18" smashed="yes">
 <attribute name="VALUE" x="203.835" y="173.355" size="1.778" layer="96"/>
@@
 <wire x1="205.74" y1="162.56" x2="205.74" y2="160.02" width="0.1524" layer="91"/>
 <pinref part="M2" gate="G$1" pin="2"/>
-<wire x1="205.74" y1="162.56" x2="220.98" y2="162.56" width="0.1524" layer="91"/>
+<wire x1="205.74" y1="162.56" x2="215.9" y2="157.48" width="0.1524" layer="91"/>
 <pinref part="VDD_12V3" gate="G$1" pin="VDD"/>
 <wire x1="205.74" y1="167.64" x2="205.74" y2="162.56" width="0.1524" layer="91"/>
@@
 <wire x1="104.14" y1="12.7" x2="104.14" y2="15.24" width="0.1524" layer="91"/>
 <label x="104.14" y="15.24" size="1.016" layer="95" rot="R90" xref="yes"/>
-<wire x1="93.98" y1="12.7" x2="104.14" y2="12.7" width="0.1524" layer="91"/>
-<wire x1="91.44" y1="2.54" x2="93.98" y2="12.7" width="0.1524" layer="91"/>
 </segment>
 <segment>
@@
 <wire x1="104.14" y1="-7.62" x2="104.14" y2="-10.16" width="0.1524" layer="91"/>
 <label x="104.14" y="-10.16" size="1.016" layer="95" rot="R270" xref="yes"/>
-<wire x1="93.98" y1="-7.62" x2="104.14" y2="-7.62" width="0.1524" layer="91"/>
-<wire x1="91.44" y1="0" x2="93.98" y2="-7.62" width="0.1524" layer="91"/>
 </segment>
 <segment>
@@
 <wire x1="104.14" y1="30.48" x2="104.14" y2="27.94" width="0.1524" layer="91"/>
 <label x="104.14" y="27.94" size="1.016" layer="95" rot="R270" xref="yes"/>
-<wire x1="93.98" y1="30.48" x2="104.14" y2="30.48" width="0.1524" layer="91"/>
-<wire x1="88.9" y1="38.1" x2="93.98" y2="30.48" width="0.1524" layer="91"/>
 </segment>
 <segment>
@@
 <wire x1="104.14" y1="50.8" x2="104.14" y2="53.34" width="0.1524" layer="91"/>
 <label x="104.14" y="53.34" size="1.016" layer="95" rot="R90" xref="yes"/>
-<wire x1="93.98" y1="50.8" x2="104.14" y2="50.8" width="0.1524" layer="91"/>
-<wire x1="88.9" y1="40.64" x2="93.98" y2="50.8" width="0.1524" layer="91"/>
 </segment>
 <segment>
@@
 <segment>
 <pinref part="D4" gate="1" pin="A"/>
-<wire x1="220.98" y1="160.02" x2="205.74" y2="154.94" width="0.1524" layer="91"/>
+<wire x1="215.9" y1="154.94" x2="205.74" y2="154.94" width="0.1524" layer="91" curve="-349.454176"/>
 <pinref part="Q2" gate="G$1" pin="D"/>
 <wire x1="205.74" y1="149.86" x2="205.74" y2="154.94" width="0.1524" layer="91"/>
@@
 <wire x1="175.26" y1="71.12" x2="177.8" y2="71.12" width="0.1524" layer="91"/>
 <label x="177.8" y="71.12" size="1.27" layer="95" xref="yes"/>
-</segment>
-<segment>
-<pinref part="JP1" gate="G$1" pin="10"/>
-<wire x1="68.58" y1="149.86" x2="73.66" y2="149.86" width="0.1524" layer="91"/>
-<label x="73.66" y="149.86" size="1.016" layer="95" xref="yes"/>
 </segment>
 <segment>
@@
 <junction x="244.475" y="104.14"/>
 </segment>
+<segment>
+<pinref part="U1" gate="G$1" pin="VDD3V3(1)"/>
+<wire x1="96.52" y1="81.28" x2="93.98" y2="81.28" width="0.1524" layer="91"/>
+<label x="93.98" y="81.28" size="1.27" layer="95" rot="R180" xref="yes"/>
+</segment>
+<segment>
+<pinref part="JP1" gate="G$1" pin="8"/>
+<wire x1="68.58" y1="144.78" x2="73.66" y2="144.78" width="0.1524" layer="91"/>
+<label x="73.66" y="144.78" size="1.016" layer="95" xref="yes"/>
+</segment>
 </net>
 <net name="A0" class="0">
@@
 <label x="73.66" y="106.68" size="1.778" layer="95"/>
 </segment>
+<segment>
+<pinref part="U$5" gate="G$1" pin="SCK"/>
+<wire x1="231.775" y1="80.01" x2="219.075" y2="80.01" width="0.1524" layer="91"/>
+<label x="220.345" y="80.01" size="1.778" layer="95"/>
+</segment>
 </net>
 <net name="EN" class="0">
@@
 </segment>
 <segment>
-<pinref part="JP1" gate="G$1" pin="8"/>
-<wire x1="68.58" y1="144.78" x2="73.66" y2="144.78" width="0.1524" layer="91"/>
-<label x="73.66" y="144.78" size="1.016" layer="95" xref="yes"/>
+<pinref part="JP1" gate="G$1" pin="9"/>
+<wire x1="68.58" y1="147.32" x2="73.66" y2="147.32" width="0.1524" layer="91"/>
+<label x="73.66" y="147.32" size="1.016" layer="95" xref="yes"/>
 </segment>
 </net>
@@
 </segment>
 <segment>
-<pinref part="JP1" gate="G$1" pin="9"/>
-<wire x1="68.58" y1="147.32" x2="73.66" y2="147.32" width="0.1524" layer="91"/>
-<label x="73.66" y="147.32" size="1.016" layer="95" xref="yes"/>
-</segment>
-<segment>
 <pinref part="SV1" gate="1" pin="5"/>
 <wire x1="71.12" y1="109.22" x2="73.66" y2="109.22" width="0.1524" layer="91"/>
@@
 <label x="220.345" y="72.39" size="1.778" layer="95"/>
 </segment>
+<segment>
+<pinref part="U1" gate="G$1" pin="RESV"/>
+<wire x1="96.52" y1="101.6" x2="93.98" y2="101.6" width="0.1524" layer="91"/>
+<label x="93.98" y="101.6" size="1.27" layer="95" rot="R180" xref="yes"/>
+</segment>
+<segment>
+<pinref part="JP1" gate="G$1" pin="10"/>
+<wire x1="68.58" y1="149.86" x2="73.66" y2="149.86" width="0.1524" layer="91"/>
+<label x="73.66" y="149.86" size="1.016" layer="95" xref="yes"/>
+</segment>
 </net>
 <net name="SCK" class="0">
@@
 <wire x1="175.26" y1="81.28" x2="180.34" y2="81.28" width="0.1524" layer="91"/>
 <label x="180.34" y="81.28" size="1.016" layer="95" xref="yes"/>
-</segment>
-<segment>
-<pinref part="U$5" gate="G$1" pin="SCK"/>
-<wire x1="231.775" y1="80.01" x2="219.075" y2="80.01" width="0.1524" layer="91"/>
-<label x="220.345" y="80.01" size="1.778" layer="95"/>
 </segment>
 </net>
@@
 <wire x1="104.14" y1="-45.72" x2="104.14" y2="-48.26" width="0.1524" layer="91"/>
 <label x="104.14" y="-48.26" size="1.016" layer="95" rot="R270" xref="yes"/>
-<wire x1="93.98" y1="-45.72" x2="104.14" y2="-45.72" width="0.1524" layer="91"/>
-<wire x1="91.44" y1="-38.1" x2="93.98" y2="-45.72" width="0.1524" layer="91"/>
 </segment>
 </net>
@@
 <wire x1="104.14" y1="-25.4" x2="104.14" y2="-22.86" width="0.1524" layer="91"/>
 <label x="104.14" y="-22.86" size="1.016" layer="95" rot="R90" xref="yes"/>
-<wire x1="93.98" y1="-25.4" x2="104.14" y2="-25.4" width="0.1524" layer="91"/>
-<wire x1="91.44" y1="-35.56" x2="93.98" y2="-25.4" width="0.1524" layer="91"/>
 </segment>
 </net>
@@
 </segment>
 <segment>
+<pinref part="U1" gate="G$1" pin="D4_-_GPIO2_/_TXD1"/>
+<wire x1="175.26" y1="96.52" x2="177.8" y2="96.52" width="0.1524" layer="91"/>
+<label x="177.8" y="96.52" size="1.016" layer="95" xref="yes"/>
+</segment>
+</net>
+<net name="DIO1" class="0">
+<segment>
+<pinref part="U$5" gate="G$1" pin="DIO1"/>
+<wire x1="231.775" y1="67.31" x2="219.075" y2="67.31" width="0.1524" layer="91"/>
+<label x="220.345" y="67.31" size="1.778" layer="95"/>
+</segment>
+<segment>
+<pinref part="U1" gate="G$1" pin="D3_-_GPIO0"/>
+<wire x1="175.26" y1="99.06" x2="177.8" y2="99.06" width="0.1524" layer="91"/>
+<label x="177.8" y="99.06" size="1.016" layer="95" xref="yes"/>
+</segment>
+</net>
+<net name="DIO2" class="0">
+<segment>
+<pinref part="U$5" gate="G$1" pin="DIO2"/>
+<wire x1="257.175" y1="72.39" x2="264.795" y2="72.39" width="0.1524" layer="91"/>
+<label x="258.445" y="72.39" size="1.778" layer="95"/>
+</segment>
+<segment>
 <pinref part="U1" gate="G$1" pin="D2_-_GPIO4"/>
 <wire x1="175.26" y1="101.6" x2="177.8" y2="101.6" width="0.1524" layer="91"/>
 <label x="177.8" y="101.6" size="1.016" layer="95" xref="yes"/>
-</segment>
-</net>
-<net name="DIO1" class="0">
-<segment>
-<pinref part="U$5" gate="G$1" pin="DIO1"/>
-<wire x1="231.775" y1="67.31" x2="219.075" y2="67.31" width="0.1524" layer="91"/>
-<label x="220.345" y="67.31" size="1.778" layer="95"/>
-</segment>
-<segment>
-<pinref part="U1" gate="G$1" pin="D3_-_GPIO0"/>
-<wire x1="175.26" y1="99.06" x2="177.8" y2="99.06" width="0.1524" layer="91"/>
-<label x="177.8" y="99.06" size="1.016" layer="95" xref="yes"/>
-</segment>
-</net>
-<net name="DIO2" class="0">
-<segment>
-<pinref part="U$5" gate="G$1" pin="DIO2"/>
-<wire x1="257.175" y1="72.39" x2="264.795" y2="72.39" width="0.1524" layer="91"/>
-<label x="258.445" y="72.39" size="1.778" layer="95"/>
-</segment>
-<segment>
-<pinref part="U1" gate="G$1" pin="D4_-_GPIO2_/_TXD1"/>
-<wire x1="175.26" y1="96.52" x2="177.8" y2="96.52" width="0.1524" layer="91"/>
-<label x="177.8" y="96.52" size="1.016" layer="95" xref="yes"/>
 </segment>
 </net>
@@
 </segment>
 </net>
-<net name="N$1" class="0">
-<segment>
-<pinref part="U1" gate="G$1" pin="RESV"/>
-<wire x1="96.52" y1="101.6" x2="93.98" y2="101.6" width="0.1524" layer="91"/>
-<label x="93.98" y="101.6" size="1.27" layer="95" rot="R180" xref="yes"/>
-</segment>
-</net>
