File: BBQ_Blower.sch (EAGLE design)
At the start: 30 parts, among them IC1 MAX31855RASA+, IC2 MAX31855RASA+, IC3 MAX31855RASA+, J3 PCC-SMP-K-100-R-ROHS, J4 PCC-SMP-K-100-R-ROHS, K1 SRD-12VDC-SL-C, K2 SRD-12VDC-SL-C, Q1 BUZ10, Q2 BUZ10, T1 2N3904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

Commit message: added Lora Component
Parts:
- removed C4: (no value), capacitor-wima:C2,5-3
- added C5: 10uF, _c2h:CAP0805-CAP-LARGEPADS
- added C6, C7: 1uF, _c2h:CAP0805-CAP-LARGEPADS
- added J$2: ANTENNATINY, _c2h:ANTENNATINY
- added TH2, TH3: (no value), SparkFun-Connectors:CONN_025MM
- added U$5: RFM95, _c2h:RFM95
- C1, C2: value (none) -> 1uF; device capacitor-wima:C2,5-3 -> _c2h:CAP0805-CAP-LARGEPADS
Connections:
- new net ANT: J$2.SIGNAL, U$5.ANT
- new net CS_LORA: U$5.SEL, U1.D12_-_GPIO10_/_SD_D3
- new net DIO0: U$5.DIO0
- new net DIO1: U$5.DIO1
- new net DIO2: U$5.DIO2
- new net GPIO12: U$5.MISO
- new net GPIO13: U$5.MOSI
- new net GPIO14: U$5.SCK
- net 3V3: now also C5.2, C6.2, C7.2, U$5.VCC; no longer C4.2
- net D3: no longer U1.D12_-_GPIO10_/_SD_D3
- net GND: now also C5.1, C6.1, C7.1, J$2.GND@0, J$2.GND@1, J$2.GND@2, J$2.GND@3, U$5.GND; no longer C4.1
- net RST: now also U$5.RST
- net T1+: now also TH3.1
- net T1-: now also TH3.2
- net T2+: now also TH2.1
- net T2-: now also TH2.2
Other:
- note added: "868MHz"
- note added: "MISO"
- note added: "MOSI"
- note added: "SCK"
- note added: "SS"
- moved on the sheet: C1, C2

Commit message: Removed Relay
Parts:
- removed D1, D2: 1N4004, adafruit:1N4004
- removed K1, K2: SRD-12VDC-SL-C, SRD-12VDC-SL-C:SRD-12VDC-SL-C
- removed R1, R2: (no value), resistor:R-US_0207/7
- removed RL1, RL2: (no value), SparkFun-Connectors:CONN_025MM
- removed T1, T2: 2N3904, transistor:2N3904
- added J1: PCC-SMP-K-100-R-ROHS, PCC-SMP-K-100-R-ROHS:PCC-SMP-K-100-R-ROHS
Connections:
- net GPIO13 renamed SI
- removed net GPIO12: U$5.MISO
- removed net GPIO14: U$5.SCK
- removed net N$1: R1.2, T2.B
- removed net N$2: D1.A, K2.3, T2.C
- removed net N$3: R2.2, T1.B
- removed net N$8: D2.A, K1.3, T1.C
- removed net RELAY1(+): K1.4, RL2.1
- removed net RELAY1(-): K1.1, RL2.2
- removed net RELAY2(+): K2.4, RL1.1
- removed net RELAY2(-): K2.1, RL1.2
- net CS_1: now also U1.D6_-_GPIO12_/_HSPIQ; no longer U1.D9_-__RXD0_/_GPIO3
- net CS_3: now also U1.D10_-_TXD0_/_GPIO1; no longer U1.D6_-_GPIO12_/_HSPIQ
- net GND: no longer T1.E, T2.E
- net RELAY_1: no longer R2.1
- net RELAY_2: no longer R1.1
- net SCK: now also U$5.SCK
- net SO: now also U$5.MISO, U1.D9_-__RXD0_/_GPIO3; no longer U1.D10_-_TXD0_/_GPIO1
- net T1+: now also TH3.2; no longer TH3.1
- net T1-: now also TH3.1; no longer TH3.2
- net T3+: now also J1.+
- net T3-: now also J1.-
- net VDD: no longer D1.C, D2.C, K1.2, K2.2

Commit message: traces
Connections:
- net T2+: now also TH2.2; no longer TH2.1
- net T2-: now also TH2.1; no longer TH2.2
- net T3+: now also TH1.2; no longer TH1.1
- net T3-: now also TH1.1; no longer TH1.2
Other:
- moved on the sheet: TH1, TH2
Changed lines of the file:
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@@
 <attribute name="VALUE" x="147.32" y="-30.48" size="1.778" layer="96" rot="R180"/>
 </instance>
-<instance part="TH1" gate="G$1" x="66.04" y="-38.1"/>
+<instance part="TH1" gate="G$1" x="81.28" y="-33.02" rot="R180"/>
 <instance part="SV1" gate="1" x="63.5" y="106.68">
 <attribute name="VALUE" x="59.69" y="99.06" size="1.778" layer="96"/>
@@
 <attribute name="VALUE" x="118.999" y="-37.211" size="1.778" layer="96" rot="R90"/>
 </instance>
-<instance part="TH2" gate="G$1" x="66.04" y="0"/>
+<instance part="TH2" gate="G$1" x="78.74" y="5.08" rot="R180"/>
 <instance part="TH3" gate="G$1" x="81.28" y="40.64" rot="R180"/>
 <instance part="J1" gate="G$1" x="104.14" y="-45.72" rot="R90">
@@
 <wire x1="83.82" y1="12.7" x2="83.82" y2="15.24" width="0.1524" layer="91"/>
 <label x="83.82" y="15.24" size="1.016" layer="95" rot="R90" xref="yes"/>
-<pinref part="TH2" gate="G$1" pin="2"/>
-<wire x1="73.66" y1="2.54" x2="73.66" y2="12.7" width="0.1524" layer="91"/>
-<wire x1="73.66" y1="12.7" x2="83.82" y2="12.7" width="0.1524" layer="91"/>
+<wire x1="71.12" y1="12.7" x2="83.82" y2="12.7" width="0.1524" layer="91"/>
+<pinref part="TH2" gate="G$1" pin="1"/>
+<wire x1="71.12" y1="5.08" x2="71.12" y2="12.7" width="0.1524" layer="91"/>
 </segment>
 </net>
@@
 <wire x1="83.82" y1="-7.62" x2="83.82" y2="-10.16" width="0.1524" layer="91"/>
 <label x="83.82" y="-10.16" size="1.016" layer="95" rot="R270" xref="yes"/>
-<pinref part="TH2" gate="G$1" pin="1"/>
-<wire x1="73.66" y1="0" x2="73.66" y2="-7.62" width="0.1524" layer="91"/>
-<wire x1="73.66" y1="-7.62" x2="83.82" y2="-7.62" width="0.1524" layer="91"/>
+<wire x1="71.12" y1="-7.62" x2="83.82" y2="-7.62" width="0.1524" layer="91"/>
+<pinref part="TH2" gate="G$1" pin="2"/>
+<wire x1="71.12" y1="-7.62" x2="71.12" y2="2.54" width="0.1524" layer="91"/>
 </segment>
 </net>
@@
 <wire x1="83.82" y1="-45.72" x2="83.82" y2="-48.26" width="0.1524" layer="91"/>
 <label x="83.82" y="-48.26" size="1.016" layer="95" rot="R270" xref="yes"/>
-<pinref part="TH1" gate="G$1" pin="1"/>
-<wire x1="73.66" y1="-38.1" x2="73.66" y2="-45.72" width="0.1524" layer="91"/>
 <wire x1="73.66" y1="-45.72" x2="83.82" y2="-45.72" width="0.1524" layer="91"/>
+<pinref part="TH1" gate="G$1" pin="2"/>
+<wire x1="73.66" y1="-45.72" x2="73.66" y2="-35.56" width="0.1524" layer="91"/>
 </segment>
 <segment>
@@
 <wire x1="83.82" y1="-25.4" x2="83.82" y2="-22.86" width="0.1524" layer="91"/>
 <label x="83.82" y="-22.86" size="1.016" layer="95" rot="R90" xref="yes"/>
-<pinref part="TH1" gate="G$1" pin="2"/>
-<wire x1="73.66" y1="-35.56" x2="73.66" y2="-25.4" width="0.1524" layer="91"/>
 <wire x1="73.66" y1="-25.4" x2="83.82" y2="-25.4" width="0.1524" layer="91"/>
-</segment>
-<segment>
+<pinref part="TH1" gate="G$1" pin="1"/>
+<wire x1="73.66" y1="-33.02" x2="73.66" y2="-25.4" width="0.1524" layer="91"/>
+</segment>
+<segment>

Commit message: restructured files
Parts:
- removed M1, M2, PWR: (no value), SparkFun-Connectors:CONN_025MM
- removed SV1: (no value), con-lstb:MA03-2
- removed U1: 113990105, 113990105:113990105
- added BLOWER1, BLOWER2, POWER, SWITCH: JST-PH_2-PIN_HEADER, SRG:JST-PH_2-PIN_HEADER
- added ICSP: (no value), con-lstb:MA03-2
- added NODE-MCU: 113990105, 113990105:113990105
- added OLED: JST-PH_4-PIN_HEADER, SRG:JST-PH_4-PIN_HEADER
- C1, C2, C5, C6, C7: device _c2h:CAP0805-CAP-LARGEPADS -> resistor:C-EUC0805K
- C3: value (none) -> 10uF; device adafruit:C-US025-060X050 -> resistor:C-EU025-050X050
Connections:
- removed net CS_1: IC1.!CS, U1.D6_-_GPIO12_/_HSPIQ
- removed net CS_2: IC2.!CS, U1.D7_-_GPIO13_/_RXD2_/_HSPID
- removed net CS_3: IC3.!CS, U1.D10_-_TXD0_/_GPIO1
- removed net RELAY_1: U1.D2_-_GPIO4
- removed net RELAY_2: U1.D3_-_GPIO0
- removed net SCK: IC1.SCK, IC2.SCK, IC3.SCK, U$5.SCK, U1.D8_-_GPIO15_/_TXD2_/_HSPICS
- removed net SI: U$5.MOSI
- removed net SO: IC1.SO, IC2.SO, IC3.SO, U$5.MISO, U1.D9_-__RXD0_/_GPIO3
- removed net SO_1: U1.D5_-_GPIO14_/_HSPICLK
- new net CS_BBQ: IC3.!CS, NODE-MCU.D10_-_TXD0_/_GPIO1
- new net CS_TF1: IC1.!CS, NODE-MCU.D9_-__RXD0_/_GPIO3
- new net CS_TF2: IC2.!CS, NODE-MCU.D8_-_GPIO15_/_TXD2_/_HSPICS
- new net DIO5: U$5.DIO5
- new net HMISO: IC1.SO, IC2.SO, IC3.SO, NODE-MCU.D6_-_GPIO12_/_HSPIQ
- new net HMOSI: NODE-MCU.D7_-_GPIO13_/_RXD2_/_HSPID
- new net HSCK: IC1.SCK, IC2.SCK, IC3.SCK, NODE-MCU.D5_-_GPIO14_/_HSPICLK
- new net SCL: NODE-MCU.D1_-_GPIO5, OLED.3
- new net SDA: NODE-MCU.D2_-_GPIO4, OLED.4
- new net VIN: POWER.1, SWITCH.1
- net 3V3: now also ICSP.6, JP1.8, NODE-MCU.VDD3V3(1), NODE-MCU.VDD3V3(2), NODE-MCU.VDD3V3(3), OLED.2; no longer JP1.10, SV1.6, U1.VDD3V3(2), U1.VDD3V3(3)
- net A0: now also NODE-MCU.A0_-_ADC_EX; no longer U1.A0_-_ADC_EX
- net BLOWER1: now also BLOWER2.2; no longer M2.1
- net BLOWER2: now also BLOWER1.2; no longer M1.1
- net BLOWER_1: now also NODE-MCU.D0_-_GPIO16; no longer U1.D0_-_GPIO16
- net BLOWER_2: now also NODE-MCU.D4_-_GPIO2_/_TXD1; no longer U1.D1_-_GPIO5
- net CLK: now also ICSP.3, NODE-MCU.SPI_CLK_/_SD_CLK, U$5.SCK; no longer SV1.3, U1.SPI_CLK_/_SD_CLK
- net CS_LORA: now also NODE-MCU.D12_-_GPIO10_/_SD_D3; no longer U1.D12_-_GPIO10_/_SD_D3
- net D1: no longer U1.SPI_INT_/_SD_D1
- net D2: no longer U1.D11_-_GPIO9_/_SD_D2
- net D4: no longer U1.D4_-_GPIO2_/_TXD1
- net DIO0: now also NODE-MCU.D11_-_GPIO9_/_SD_D2
- net DIO1: now also NODE-MCU.D3_-_GPIO0
- net EN: now also JP1.9, NODE-MCU.EN; no longer JP1.8, U1.EN
- net GND: now also ICSP.2, NODE-MCU.GND(1), NODE-MCU.GND(2), NODE-MCU.GND(3), NODE-MCU.GND(4), OLED.1, POWER.2; no longer PWR.1, SV1.2, U1.GND(2), U1.GND(3)
- net MISO: now also ICSP.1, NODE-MCU.SPI_MISO_/_SD_D0, U$5.MISO; no longer SV1.1, U1.SPI_MISO_/_SD_D0
- net MOSI: now also ICSP.4, NODE-MCU.SPI_INT_/_SD_D1, NODE-MCU.SPI_MOSI_/_SD_CMD, U$5.MOSI; no longer SV1.4, U1.SPI_MOSI_/_SD_CMD
- net RST: now also ICSP.5, JP1.10, NODE-MCU.NRST; no longer JP1.9, SV1.5, U1.NRST
- net VDD: now also BLOWER1.1, BLOWER2.1, NODE-MCU.VDD5V, SWITCH.2; no longer M1.2, M2.2, PWR.2, U1.VDD5V
Other:
- note added: "Board: BBQ Controller Author: Cody Fischer Date: August 2019 Rev: 1.0"
- note removed: "MISO"
- note removed: "MOSI"
- note removed: "SCK"
- note removed: "SS"
- moved on the sheet: C1, C2, C3, C5, C6, C7, D3, D4, IC1, IC2, IC3, J1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

Commit message: first final
Parts:
- added R1, R2: 4.7K, _c2h:RESISTOR0805-RES
Connections:
- net 3V3: now also R1.2, R2.2
- net SCL: now also R1.1
- net SDA: now also R2.1
Changed lines of the file:
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@@
 </variantdefs>
 <classes>
-<class number="0" name="default" width="0.3048" drill="0.3556">
-<clearance class="0" value="0.254"/>
+<class number="0" name="default" width="0.2032" drill="0.3556">
+<clearance class="0" value="0.1524"/>
 </class>
 <class number="1" name="POWER" width="1.905" drill="0">
@@
 <part name="OLED" library="SRG" deviceset="JST-PH_4-PIN_HEADER" device=""/>
 <part name="SWITCH" library="SRG" deviceset="JST-PH_2-PIN_HEADER" device=""/>
+<part name="R1" library="_c2h" deviceset="RESISTOR" device="0805-RES" value="4.7K"/>
+<part name="R2" library="_c2h" deviceset="RESISTOR" device="0805-RES" value="4.7K"/>
+<part name="+3V2" library="supply1" deviceset="+3V3" device=""/>
 </parts>
 <sheets>
@@
 <attribute name="VALUE" x="99.06" y="122.682" size="1.27" layer="96" font="vector"/>
 </instance>
+<instance part="R1" gate="G$1" x="86.995" y="88.9" smashed="yes" rot="R90">
+<attribute name="NAME" x="85.4964" y="90.17" size="1.778" layer="95" rot="R90"/>
+<attribute name="VALUE" x="90.297" y="85.09" size="1.778" layer="96" rot="R90"/>
+</instance>
+<instance part="R2" gate="G$1" x="79.375" y="86.36" smashed="yes" rot="R90">
+<attribute name="NAME" x="77.8764" y="85.09" size="1.778" layer="95" rot="R90"/>
+<attribute name="VALUE" x="82.677" y="82.55" size="1.778" layer="96" rot="R90"/>
+</instance>
+<instance part="+3V2" gate="G$1" x="69.215" y="99.06" smashed="yes">
+<attribute name="VALUE" x="71.755" y="101.6" size="1.778" layer="96" rot="R180"/>
+</instance>
 </instances>
 <busses>
@@
 <label x="93.98" y="86.36" size="1.778" layer="95"/>
 </segment>
+<segment>
+<pinref part="R2" gate="G$1" pin="2"/>
+<wire x1="79.375" y1="91.44" x2="68.58" y2="91.44" width="0.1524" layer="91"/>
+<pinref part="+3V2" gate="G$1" pin="+3V3"/>
+<wire x1="68.58" y1="91.44" x2="68.58" y2="96.52" width="0.1524" layer="91"/>
+<wire x1="68.58" y1="96.52" x2="69.215" y2="96.52" width="0.1524" layer="91"/>
+<pinref part="R1" gate="G$1" pin="2"/>
+<wire x1="86.995" y1="93.98" x2="71.12" y2="93.98" width="0.1524" layer="91"/>
+<wire x1="71.12" y1="93.98" x2="71.12" y2="96.52" width="0.1524" layer="91"/>
+<wire x1="71.12" y1="96.52" x2="69.215" y2="96.52" width="0.1524" layer="91"/>
+<junction x="69.215" y="96.52"/>
+<label x="76.2" y="93.98" size="1.778" layer="95"/>
+</segment>
 </net>
 <net name="A0" class="0">
@@
 </segment>
 <segment>
-<wire x1="99.06" y1="83.82" x2="93.98" y2="83.82" width="0.1524" layer="91"/>
 <pinref part="OLED" gate="G$1" pin="3"/>
 <label x="93.98" y="83.82" size="1.778" layer="95"/>
+<pinref part="R1" gate="G$1" pin="1"/>
+<wire x1="99.06" y1="83.82" x2="86.995" y2="83.82" width="0.1524" layer="91"/>
 </segment>
 </net>
@@
 </segment>
 <segment>
-<wire x1="99.06" y1="81.28" x2="93.98" y2="81.28" width="0.1524" layer="91"/>
 <pinref part="OLED" gate="G$1" pin="4"/>
 <label x="93.98" y="81.28" size="1.778" layer="95"/>
-</segment>
-</net>
+<pinref part="R2" gate="G$1" pin="1"/>
+<wire x1="99.06" y1="81.28" x2="79.375" y2="81.28" width="0.1524" layer="91"/>
+<wire x1="79.375" y1="81.28" x2="78.74" y2="81.28" width="0.1524" layer="91"/>
+<junction x="79.375" y="81.28"/>
+</segment>
+</net>
